Commit message: Update differential drive plugin & friction params

File: my_rb1_description/urdf/my_rb1_robot.urdf (robot description, URDF)
Before this commit: robot rb1_robot_kailash, 7 links, 6 joints
Joints:
- joint joint_base_left_wheel: limit effort=10000 velocity=1000 -> (none)
- joint joint_base_right_wheel: limit effort=10000 velocity=1000 -> (none)
